Commit message: Add UR5 robot description and cleanup script
- Created a new URDF/Xacro file for the UR5 robot with RG2 gripper, including joint definitions and ros2_control configuration.
- Added a script to clean up the ROS 2 stack, handling process termination and shared memory cleanup.
- Introduced a wrapper script to execute the cleanup script from a different location.

File: agarre_ros2_ws/backups/before_sdf_prismatic_fix/urdf/ur5.urdf.xacro (robot description, xacro)
@@ -42,20 +42,11 @@
     <origin xyz="-0.85 0 0.850" rpy="0 0 0"/>
   </xacro:ur_robot>
-  <!-- RG2 gripper: simplified prismatic box geometry, coherent with SDF/TF/ros2_control. -->
+  <!-- RG2 gripper (simplified kinematic stub for ros2_control) -->
   <link name="rg2_base_link">
     <inertial>
-      <mass value="0.30"/>
-      <origin xyz="0 0 0.010" rpy="0 0 0"/>
-      <inertia ixx="0.00050" ixy="0.0" ixz="0.0" iyy="0.00040" iyz="0.0" izz="0.00060"/>
+      <mass value="0.5"/>
+      <origin xyz="0 0 0" rpy="0 0 0"/>
+      <inertia ixx="0.001" ixy="0.0" ixz="0.0" iyy="0.001" iyz="0.0" izz="0.001"/>
     </inertial>
-    <visual>
-      <origin xyz="0 0 0.010" rpy="0 0 0"/>
-      <geometry><box size="0.060 0.080 0.020"/></geometry>
-      <material name="rg2_gray"><color rgba="0.4 0.4 0.4 1"/></material>
-    </visual>
-    <collision>
-      <origin xyz="0 0 0.010" rpy="0 0 0"/>
-      <geometry><box size="0.060 0.080 0.020"/></geometry>
-    </collision>
   </link>
   <joint name="rg2_mount_joint" type="fixed">
@@ -95,51 +86,31 @@
     <origin xyz="${rg2_contact_tcp_xyz}" rpy="0 0 0"/>
   </joint>
-  <!-- Finger links: box 12x10x175 mm; joint origin at ±20 mm Y from rg2_base_link. -->
-  <!-- Visual center at 0 0 0.0875 (half of 175 mm) in finger-link frame. -->
   <link name="rg2_finger_link1">
     <inertial>
       <mass value="0.05"/>
-      <origin xyz="0 0 0.0875" rpy="0 0 0"/>
-      <inertia ixx="1.3e-4" ixy="0.0" ixz="0.0" iyy="1.3e-4" iyz="0.0" izz="1.0e-6"/>
+      <origin xyz="0 0 0" rpy="0 0 0"/>
+      <inertia ixx="1e-4" ixy="0.0" ixz="0.0" iyy="1e-4" iyz="0.0" izz="1e-4"/>
     </inertial>
-    <visual>
-      <origin xyz="0 0 0.0875" rpy="0 0 0"/>
-      <geometry><box size="0.012 0.010 0.175"/></geometry>
-      <material name="rg2_dark_gray"><color rgba="0.25 0.25 0.25 1"/></material>
-    </visual>
-    <collision>
-      <origin xyz="0 0 0.0875" rpy="0 0 0"/>
-      <geometry><box size="0.012 0.010 0.175"/></geometry>
-    </collision>
   </link>
   <link name="rg2_finger_link2">
     <inertial>
       <mass value="0.05"/>
-      <origin xyz="0 0 0.0875" rpy="0 0 0"/>
-      <inertia ixx="1.3e-4" ixy="0.0" ixz="0.0" iyy="1.3e-4" iyz="0.0" izz="1.0e-6"/>
+      <origin xyz="0 0 0" rpy="0 0 0"/>
+      <inertia ixx="1e-4" ixy="0.0" ixz="0.0" iyy="1e-4" iyz="0.0" izz="1e-4"/>
     </inertial>
-    <visual>
-      <origin xyz="0 0 0.0875" rpy="0 0 0"/>
-      <geometry><box size="0.012 0.010 0.175"/></geometry>
-      <material name="rg2_dark_gray"/>
-    </visual>
-    <collision>
-      <origin xyz="0 0 0.0875" rpy="0 0 0"/>
-      <geometry><box size="0.012 0.010 0.175"/></geometry>
-    </collision>
   </link>
   <joint name="rg2_finger_joint1" type="prismatic">
     <parent link="rg2_base_link"/>
     <child link="rg2_finger_link1"/>
-    <origin xyz="0 0.020 0" rpy="0 0 0"/>
+    <origin xyz="0 0.02 0" rpy="0 0 0"/>
     <axis xyz="0 1 0"/>
-    <limit lower="0.0" upper="0.0425" effort="20" velocity="0.2"/>
+    <limit lower="0.0" upper="0.04" effort="20" velocity="0.2"/>
   </joint>
   <joint name="rg2_finger_joint2" type="prismatic">
     <parent link="rg2_base_link"/>
     <child link="rg2_finger_link2"/>
-    <origin xyz="0 -0.020 0" rpy="0 0 0"/>
+    <origin xyz="0 -0.02 0" rpy="0 0 0"/>
     <axis xyz="0 -1 0"/>
-    <limit lower="0.0" upper="0.0425" effort="20" velocity="0.2"/>
+    <limit lower="0.0" upper="0.04" effort="20" velocity="0.2"/>
   </joint>
   <!-- ros2_control (gz_ros2_control) with UR5 + RG2 joints -->
