Commit message: Restructure workspace and regenerate chapter 5 artifacts

File: agarre_ros2_ws/src/ur5_description/urdf/ur5.urdf.xacro (robot description, xacro)
@@ -33,5 +33,5 @@
     force_abs_paths="${force_abs_paths}"
     >
-    <origin xyz="-0.85 0 0.775" rpy="0 0 0"/>
+    <origin xyz="-0.85 0 0.825" rpy="0 0 0"/>
   </xacro:ur_robot>
   <!-- RG2 gripper (simplified kinematic stub for ros2_control) -->
@@ -96,40 +96,56 @@
     <joint name="shoulder_pan_joint">
       <command_interface name="position"/>
-      <state_interface name="position"/>
+      <state_interface name="position">
+        <param name="initial_value">0.0</param>
+      </state_interface>
       <state_interface name="velocity"/>
     </joint>
     <joint name="shoulder_lift_joint">
       <command_interface name="position"/>
-      <state_interface name="position"/>
+      <state_interface name="position">
+        <param name="initial_value">-1.5707963267948966</param>
+      </state_interface>
       <state_interface name="velocity"/>
     </joint>
     <joint name="elbow_joint">
       <command_interface name="position"/>
-      <state_interface name="position"/>
+      <state_interface name="position">
+        <param name="initial_value">0.0</param>
+      </state_interface>
       <state_interface name="velocity"/>
     </joint>
     <joint name="wrist_1_joint">
       <command_interface name="position"/>
-      <state_interface name="position"/>
+      <state_interface name="position">
+        <param name="initial_value">-1.5707963267948966</param>
+      </state_interface>
       <state_interface name="velocity"/>
     </joint>
     <joint name="wrist_2_joint">
       <command_interface name="position"/>
-      <state_interface name="position"/>
+      <state_interface name="position">
+        <param name="initial_value">0.0</param>
+      </state_interface>
       <state_interface name="velocity"/>
     </joint>
     <joint name="wrist_3_joint">
       <command_interface name="position"/>
-      <state_interface name="position"/>
+      <state_interface name="position">
+        <param name="initial_value">0.0</param>
+      </state_interface>
       <state_interface name="velocity"/>
     </joint>
     <joint name="rg2_finger_joint1">
       <command_interface name="position"/>
-      <state_interface name="position"/>
+      <state_interface name="position">
+        <param name="initial_value">0.0</param>
+      </state_interface>
       <state_interface name="velocity"/>
     </joint>
     <joint name="rg2_finger_joint2">
       <command_interface name="position"/>
-      <state_interface name="position"/>
+      <state_interface name="position">
+        <param name="initial_value">0.0</param>
+      </state_interface>
       <state_interface name="velocity"/>
     </joint>

Commit message: Añadir imagen superpuesta con los resultados de inferencia en la auditoría del panel.

File: agarre_ros2_ws/src/ur5_description/urdf/ur5.urdf.xacro (robot description, xacro)
@@ -59,5 +59,5 @@
     <parent link="tool0"/>
     <child link="rg2_tcp"/>
-    <origin xyz="0 0 0.23" rpy="0 0 0"/>
+    <origin xyz="0 0 0.175" rpy="0 0 0"/>
   </joint>
   <link name="rg2_finger_link1">

Commit message: Actualizar los artefactos de auditoría de MoveIt y añadir una nueva imagen de superposición 	•	Se modificó tfm_moveit_canonical_last.json para reflejar los nuevos detalles de la sesión y el objeto seleccionado. 	•	Se actualizaron los parámetros base del agarre, incluida la posición y su semántica. 	•	Se ajustaron las marcas temporales y los detalles de los eventos para que coincidan con el contexto de ejecución más reciente. 	•	Se sustituyó la imagen existente overlay_last.png por una versión actualizada. 	•	Se añadió la nueva imagen de superposición overlay_infer_61288632.png para la visualización de la inferencia.

File: agarre_ros2_ws/src/ur5_description/urdf/ur5.urdf.xacro (robot description, xacro)
@@ -60,4 +60,19 @@
     <child link="rg2_tcp"/>
     <origin xyz="0 0 0.175" rpy="0 0 0"/>
+  </joint>
+  <!-- Operational pinch-center: midpoint between the two RG2 fingers in this
+       simplified kinematic model. The prismatic fingers are symmetric about
+       rg2_base_link/tool0, so their functional midpoint lives at tool0. -->
+  <link name="rg2_pinch_center">
+    <inertial>
+      <mass value="0.01"/>
+      <origin xyz="0 0 0" rpy="0 0 0"/>
+      <inertia ixx="1e-5" ixy="0.0" ixz="0.0" iyy="1e-5" iyz="0.0" izz="1e-5"/>
+    </inertial>
+  </link>
+  <joint name="rg2_pinch_center_joint" type="fixed">
+    <parent link="tool0"/>
+    <child link="rg2_pinch_center"/>
+    <origin xyz="0 0 0" rpy="0 0 0"/>
   </joint>
   <link name="rg2_finger_link1">

Commit message: Añadir archivos de benchmark y trazas para la validación de DIRECTO en múltiples sesiones 	•	Se crearon los archivos benchmark.json y benchmark_stdout.json para las sesiones de validación con marcas de tiempo 113309, 114504, 120403, 125823, 131439, 135136 y 173827. 	•	Se añadieron archivos orchestrator_summary.txt para resumir los resultados de cada sesión de validación. 	•	Se introdujeron archivos directo_trace.jsonl para cada sesión, con datos de trazado; el tamaño de estos archivos es demasiado grande para mostrar un diff. 	•	Las métricas y veredictos incluidos en los archivos de benchmark reflejan el rendimiento y los resultados del modo DIRECTO.

File: agarre_ros2_ws/src/ur5_description/urdf/ur5.urdf.xacro (robot description, xacro)
@@ -61,7 +61,7 @@
     <origin xyz="0 0 0.175" rpy="0 0 0"/>
   </joint>
-  <!-- Operational pinch-center: midpoint between the two RG2 fingers in this
-       simplified kinematic model. The prismatic fingers are symmetric about
-       rg2_base_link/tool0, so their functional midpoint lives at tool0. -->
+    <!-- Operational pinch-center: contact midpoint between the two RG2 fingers.
+      In this simplified model the contact point is aligned with the same TCP
+      used at the fingertips, so it must stay offset from tool0. -->
   <link name="rg2_pinch_center">
     <inertial>
@@ -74,5 +74,5 @@
     <parent link="tool0"/>
     <child link="rg2_pinch_center"/>
-    <origin xyz="0 0 0" rpy="0 0 0"/>
+    <origin xyz="0 0 0.175" rpy="0 0 0"/>
   </joint>
   <link name="rg2_finger_link1">

Commit message: Eliminar archivos obsoletos y añadir nuevas configuraciones y modelos para SimpleGrasp 	•	Se eliminó el archivo de registro JSON desactualizado: episode_20260407_215744.json 	•	Se eliminaron los archivos de documentación de auditoría del workspace: AUDITORIA_WORKSPACE_LIMPIEZA.md, MATRIZ_WORKSPACE.csv, RESUMEN_READMES.md 	•	Se eliminaron los archivos de frames sin uso: frames_2026-04-06_23.28.39.gv, frames_2026-04-06_23.28.39.pdf 	•	Se actualizó el README del informe para reflejar las nuevas rutas de logs y ejecución. 	•	Se añadieron nuevos archivos de configuración para los modelos SimpleGrasp: exp5_simplegrasp_rgb.yaml, exp6_simplegrasp_rgbd.yaml 	•	Se incorporó una factoría de modelos para construir modelos según la configuración: factory.py 	•	Se implementó la arquitectura del modelo SimpleGrasp: simple_grasp.py

File: agarre_ros2_ws/src/ur5_description/urdf/ur5.urdf.xacro (robot description, xacro)
@@ -33,5 +33,9 @@
     force_abs_paths="${force_abs_paths}"
     >
-    <origin xyz="-0.85 0 0.825" rpy="0 0 0"/>
+    <!-- Keep the URDF world origin aligned with the Gazebo world include pose.
+         If these diverge, robot_state_publisher TF and the rendered Gazebo model
+         disagree in Z, which makes the panel report a different TCP height than
+         the one visible in the simulator. -->
+    <origin xyz="-0.85 0 0.850" rpy="0 0 0"/>
   </xacro:ur_robot>
   <!-- RG2 gripper (simplified kinematic stub for ros2_control) -->

Commit message: feat: Ajusta la posición del TCP visual en rg2_tcp y corrige el offset en gripper_attach_backend.py

File: agarre_ros2_ws/src/ur5_description/urdf/ur5.urdf.xacro (robot description, xacro)
@@ -52,5 +52,8 @@
     <origin xyz="0 0 0" rpy="0 0 0"/>
   </joint>
-  <!-- Virtual TCP at the gripper fingertips (fixed offset from tool0). -->
+  <!-- Visual TCP at the gripper fingertip tips (mesh-matched offset from tool0).
+       0.213 m = finger_pivot_reach (0.105) + finger_mesh_reach (0.108),
+       derived from the finger.dae geometry — where the fingertip mesh ends.
+       rg2_pinch_center (0.175) is the operational grasp center; rg2_tcp is visual-only. -->
   <link name="rg2_tcp">
     <inertial>
@@ -63,5 +66,5 @@
     <parent link="tool0"/>
     <child link="rg2_tcp"/>
-    <origin xyz="0 0 0.175" rpy="0 0 0"/>
+    <origin xyz="0 0 0.213" rpy="0 0 0"/>
   </joint>
     <!-- Operational pinch-center: contact midpoint between the two RG2 fingers.

Commit message: feat: Ajusta offsets del TCP y gripper en SDF y URDF, añade captura de frames de cámara

File: agarre_ros2_ws/src/ur5_description/urdf/ur5.urdf.xacro (robot description, xacro)
@@ -52,8 +52,7 @@
     <origin xyz="0 0 0" rpy="0 0 0"/>
   </joint>
-  <!-- Visual TCP at the gripper fingertip tips (mesh-matched offset from tool0).
-       0.213 m = finger_pivot_reach (0.105) + finger_mesh_reach (0.108),
-       derived from the finger.dae geometry — where the fingertip mesh ends.
-       rg2_pinch_center (0.175) is the operational grasp center; rg2_tcp is visual-only. -->
+  <!-- Visual TCP: coincide con rg2_pinch_center (0.175m desde tool0) gracias al offset
+       SDF ur5_hand_joint=0.237456 que alinea las yemas del mesh con el TCP operacional.
+       Con SDF=0.237456: fingertip_wrist3 = 0.237456+0.213 = 0.450m = rg2_pinch_center. -->
   <link name="rg2_tcp">
     <inertial>
@@ -66,5 +65,5 @@
     <parent link="tool0"/>
     <child link="rg2_tcp"/>
-    <origin xyz="0 0 0.213" rpy="0 0 0"/>
+    <origin xyz="0 0 0.175" rpy="0 0 0"/>
   </joint>
     <!-- Operational pinch-center: contact midpoint between the two RG2 fingers.

Commit message: fix: ajustar offsets TCP para alineación visual precisa en el sistema UR5 con RG2

File: agarre_ros2_ws/src/ur5_description/urdf/ur5.urdf.xacro (robot description, xacro)
@@ -52,8 +52,8 @@
     <origin xyz="0 0 0" rpy="0 0 0"/>
   </joint>
-  <!-- Virtual TCP frame at the operational grasp center (0.175m from tool0).
-       SDF ur5_hand_joint=0.0823 places the rg2_hand mesh at the physical flange;
-       the visual fingertips in Gazebo appear at tool0+0.020m (cosmetic offset),
-       but this frame defines the semantic grasp point used by planning/attach. -->
+  <!-- Virtual TCP frame at the operational grasp center used by planning/attach.
+       Gazebo's visible closure midpoint lies behind tool0 in the tool local +Z axis,
+       so this semantic frame must match that visual midpoint instead of the legacy
+       +0.175 m offset. -->
   <link name="rg2_tcp">
     <inertial>
@@ -66,9 +66,9 @@
     <parent link="tool0"/>
     <child link="rg2_tcp"/>
-    <origin xyz="0 0 0.175" rpy="0 0 0"/>
+    <origin xyz="0 0 -0.0877005" rpy="0 0 0"/>
   </joint>
     <!-- Operational pinch-center: contact midpoint between the two RG2 fingers.
-      In this simplified model the contact point is aligned with the same TCP
-      used at the fingertips, so it must stay offset from tool0. -->
+      Keep it coincident with the semantic TCP so DIRECTO, MoveIt and attach all
+      reason about the same visible closure center. -->
   <link name="rg2_pinch_center">
     <inertial>
@@ -81,5 +81,5 @@
     <parent link="tool0"/>
     <child link="rg2_pinch_center"/>
-    <origin xyz="0 0 0.175" rpy="0 0 0"/>
+    <origin xyz="0 0 -0.0877005" rpy="0 0 0"/>
   </joint>
   <link name="rg2_finger_link1">

Commit message: fix: ajustar offsets TCP para alineación precisa del gripper RG2 en múltiples archivos

File: agarre_ros2_ws/src/ur5_description/urdf/ur5.urdf.xacro (robot description, xacro)
@@ -53,7 +53,7 @@
   </joint>
   <!-- Virtual TCP frame at the operational grasp center used by planning/attach.
-       Gazebo's visible closure midpoint lies behind tool0 in the tool local +Z axis,
-       so this semantic frame must match that visual midpoint instead of the legacy
-       +0.175 m offset. -->
+       The RG2 contact midpoint is slightly in front of tool0 in tool local +Z:
+       the previous -0.0877005 value landed near the finger hinges, leaving the
+       semantic TCP about 9.3 cm behind the visible pinch center. -->
   <link name="rg2_tcp">
     <inertial>
@@ -66,5 +66,5 @@
     <parent link="tool0"/>
     <child link="rg2_tcp"/>
-    <origin xyz="0 0 -0.0877005" rpy="0 0 0"/>
+    <origin xyz="0 0 0.0050885" rpy="0 0 0"/>
   </joint>
     <!-- Operational pinch-center: contact midpoint between the two RG2 fingers.
@@ -81,5 +81,5 @@
     <parent link="tool0"/>
     <child link="rg2_pinch_center"/>
-    <origin xyz="0 0 -0.0877005" rpy="0 0 0"/>
+    <origin xyz="0 0 0.0050885" rpy="0 0 0"/>
   </joint>
   <link name="rg2_finger_link1">

Commit message: fix(geometry): congelar tcp canonico rg2 y unificar frame operativo

File: agarre_ros2_ws/src/ur5_description/urdf/ur5.urdf.xacro (robot description, xacro)
@@ -14,4 +14,7 @@
   <xacro:property name="robot_name" value="ur5_rg2"/>
   <xacro:property name="tf_prefix_value" value=""/>
+  <!-- Offset operativo canónico del TCP validado el 2026-04-21.
+       No retocar sin una nueva revalidación visual. -->
+  <xacro:property name="rg2_contact_tcp_xyz" value="0 0 0.0050885"/>
   <xacro:property name="joint_limits_file" value="${ur_pkg_share}/config/${ur_type}/joint_limits.yaml"/>
   <xacro:property name="kinematics_file" value="${ur_pkg_share}/config/${ur_type}/default_kinematics.yaml"/>
@@ -66,5 +69,5 @@
     <parent link="tool0"/>
     <child link="rg2_tcp"/>
-    <origin xyz="0 0 0.0050885" rpy="0 0 0"/>
+    <origin xyz="${rg2_contact_tcp_xyz}" rpy="0 0 0"/>
   </joint>
     <!-- Operational pinch-center: contact midpoint between the two RG2 fingers.
@@ -81,5 +84,5 @@
     <parent link="tool0"/>
     <child link="rg2_pinch_center"/>
-    <origin xyz="0 0 0.0050885" rpy="0 0 0"/>
+    <origin xyz="${rg2_contact_tcp_xyz}" rpy="0 0 0"/>
   </joint>
   <link name="rg2_finger_link1">

Commit message: Fix canonical RG2 terminal geometry

File: agarre_ros2_ws/src/ur5_description/urdf/ur5.urdf.xacro (robot description, xacro)
@@ -14,7 +14,7 @@
   <xacro:property name="robot_name" value="ur5_rg2"/>
   <xacro:property name="tf_prefix_value" value=""/>
-  <!-- Offset operativo canónico del TCP validado el 2026-04-21.
-       No retocar sin una nueva revalidación visual. -->
-  <xacro:property name="rg2_contact_tcp_xyz" value="0 0 0.0050885"/>
+  <!-- Offset físico real flange→yemas: 0.175 m (ur5_hand_joint Z=0.07 + finger_joint X=0.105).
+       Corregido con Opción 3 SDF fix (2026-04-24). -->
+  <xacro:property name="rg2_contact_tcp_xyz" value="0 0 0.175"/>
   <xacro:property name="joint_limits_file" value="${ur_pkg_share}/config/${ur_type}/joint_limits.yaml"/>
   <xacro:property name="kinematics_file" value="${ur_pkg_share}/config/${ur_type}/default_kinematics.yaml"/>
