Commit message: Refactor code structure for improved readability and maintainability

File: agarre_ros2_ws/src/ur5_description/urdf/ur5.urdf.xacro (robot description, xacro)
@@ -1,9 +1,9 @@
 <?xml version="1.0"?>
 <!-- Ruta/archivo: agarre_ros2_ws/src/ur5_description/urdf/ur5.urdf.xacro -->
-<!-- Contenido: Descripcion URDF/Xacro y configuracion base del robot UR5. -->
+<!-- Contenido: Descripcion URDF/Xacro y configuracion base del robot UR5 con TCP limpio. -->
 <!-- Uso breve: Se usa al publicar el robot model y al preparar simulacion y MoveIt. -->
 <!-- URL: /home/laboratorio/TFM/agarre_ros2_ws/src/ur5_description/urdf/ur5.urdf.xacro -->
-<!-- Summary: UR5 description with mock ros2_control and RG2 gripper joints. -->
-<robot xmlns:xacro="http://wiki.ros.org/xacro" name="ur5_rg2">
+<!-- Summary: UR5 description with clean prismatic TCP (tcp_clean_link/tcp_tip). No RG2. -->
+<robot xmlns:xacro="http://wiki.ros.org/xacro" name="ur5_tcp_clean">
   <xacro:property name="ur_type" value="ur5"/>
   <xacro:property name="safety_limits" value="false"/>
@@ -12,11 +12,6 @@
   <xacro:property name="force_abs_paths" value="false"/>
   <xacro:property name="ur_pkg_share" value="$(optenv UR_DESCRIPTION_SHARE /opt/ros/jazzy/share/ur_description)"/>
-  <xacro:property name="robot_name" value="ur5_rg2"/>
+  <xacro:property name="robot_name" value="ur5_tcp_clean"/>
   <xacro:property name="tf_prefix_value" value=""/>
-  <!-- TCP semántico canónico rg2_pinch_center / rg2_tcp: 0.0050885 m desde tool0.
-       Este es el único valor válido para frames operacionales de pick, MoveIt y attach.
-       Nota: las yemas visuales de los dedos quedan a 0.120 + 0.055 = 0.175 m de tool0
-       por geometría del útil (solo relevante para visual/collision, no para TCP semántico). -->
-  <xacro:property name="rg2_contact_tcp_xyz" value="0 0 0.0050885"/>
   <xacro:property name="joint_limits_file" value="${ur_pkg_share}/config/${ur_type}/joint_limits.yaml"/>
   <xacro:property name="kinematics_file" value="${ur_pkg_share}/config/${ur_type}/default_kinematics.yaml"/>
@@ -38,118 +33,50 @@
     force_abs_paths="${force_abs_paths}"
     >
-    <!-- Keep the URDF world origin aligned with the Gazebo world include pose.
-         If these diverge, robot_state_publisher TF and the rendered Gazebo model
-         disagree in Z, which makes the panel report a different TCP height than
-         the one visible in the simulator. -->
     <origin xyz="-0.85 0 0.850" rpy="0 0 0"/>
   </xacro:ur_robot>
-  <!-- RG2 schematic gripper — geometry mirroring the visual_autopick_ros_ws reference.
-       rg2_hand      : gripper housing (box 60×80×120 mm), mounted at tool0.
-       rg2_leftfinger / rg2_rightfinger : thin box fingers (12×10×55 mm), prismatic ±Y.
-       Finger pivot at Z=0.120 from rg2_hand; visual tip at tool0 Z=0.175 (visual geometry only).
-       TCP semántico operacional (rg2_pinch_center) = rg2_contact_tcp_xyz = 0 0 0.0050885.
-         joint = 0.000 m → cerrada  (dedos centrados)
-         joint = 0.055 m → abierta  (cada dedo 55 mm del centro, 110 mm total) -->
-  <link name="rg2_hand">
-    <inertial>
-      <mass value="0.490"/>
-      <origin xyz="0 0 0.060" rpy="0 0 0"/>
-      <inertia ixx="0.0004" ixy="0.0" ixz="0.0" iyy="0.0004" iyz="0.0" izz="0.0003"/>
-    </inertial>
+  <!-- Clean prismatic TCP: box 30x30x180mm, from tool0 downward.
+       tcp_clean_link center at Z=-0.09 from tool0; tcp_tip at Z=-0.18 from tool0.
+       This is the single operational TCP frame for DIRECTO, MoveIt and pick. -->
+  <link name="tcp_clean_link">
     <visual>
-      <origin xyz="0 0 0.060" rpy="0 0 0"/>
-      <geometry><box size="0.060 0.080 0.120"/></geometry>
-      <material name="RG2Gray"><color rgba="0.18 0.18 0.18 1.0"/></material>
+      <origin xyz="0 0 -0.09" rpy="0 0 0"/>
+      <geometry>
+        <box size="0.03 0.03 0.18"/>
+      </geometry>
+      <material name="tcp_clean_blue">
+        <color rgba="0.1 0.3 1.0 1.0"/>
+      </material>
     </visual>
     <collision>
-      <origin xyz="0 0 0.060" rpy="0 0 0"/>
-      <geometry><box size="0.060 0.080 0.120"/></geometry>
+      <origin xyz="0 0 -0.09" rpy="0 0 0"/>
+      <geometry>
+        <box size="0.03 0.03 0.18"/>
+      </geometry>
     </collision>
+    <inertial>
+      <origin xyz="0 0 -0.09" rpy="0 0 0"/>
+      <mass value="0.05"/>
+      <inertia
+        ixx="0.00015"
+        ixy="0.0"
+        ixz="0.0"
+        iyy="0.00015"
+        iyz="0.0"
+        izz="0.00005"/>
+    </inertial>
   </link>
-  <joint name="rg2_mount_joint" type="fixed">
+  <joint name="tool0_to_tcp_clean_joint" type="fixed">
     <parent link="tool0"/>
-    <child link="rg2_hand"/>
+    <child link="tcp_clean_link"/>
     <origin xyz="0 0 0" rpy="0 0 0"/>
   </joint>
-  <!-- TCP alias frame: igual que rg2_pinch_center (0 0 0.0050885 desde tool0), mantenido como alias. -->
-  <link name="rg2_tcp">
-    <inertial>
-      <mass value="0.01"/>
-      <origin xyz="0 0 0" rpy="0 0 0"/>
-      <inertia ixx="1e-5" ixy="0.0" ixz="0.0" iyy="1e-5" iyz="0.0" izz="1e-5"/>
-    </inertial>
-  </link>
-  <joint name="rg2_tcp_joint" type="fixed">
-    <parent link="tool0"/>
-    <child link="rg2_tcp"/>
-    <origin xyz="${rg2_contact_tcp_xyz}" rpy="0 0 0"/>
+  <link name="tcp_tip"/>
+  <joint name="tcp_clean_to_tcp_tip_joint" type="fixed">
+    <parent link="tcp_clean_link"/>
+    <child link="tcp_tip"/>
+    <origin xyz="0 0 -0.18" rpy="0 0 0"/>
   </joint>
-  <!-- Frame operacional: 0.0050885 m desde tool0 (rg2_contact_tcp_xyz canónico).
-       TCP único usado por DIRECTO, MoveIt y el sistema attach/carry. -->
-  <link name="rg2_pinch_center">
-    <inertial>
-      <mass value="0.01"/>
-      <origin xyz="0 0 0" rpy="0 0 0"/>
-      <inertia ixx="1e-5" ixy="0.0" ixz="0.0" iyy="1e-5" iyz="0.0" izz="1e-5"/>
-    </inertial>
-  </link>
-  <joint name="rg2_pinch_center_joint" type="fixed">
-    <parent link="tool0"/>
-    <child link="rg2_pinch_center"/>
-    <origin xyz="${rg2_contact_tcp_xyz}" rpy="0 0 0"/>
-  </joint>
-  <!-- Left finger: caja 12×10×55 mm, pivote en Z=0.120 desde rg2_hand.
-       Yema visual en Z=0.175 desde tool0 (solo geometría visual, no TCP semántico). -->
-  <link name="rg2_leftfinger">
-    <inertial>
-      <mass value="0.040"/>
-      <origin xyz="0 0 0.0275" rpy="0 0 0"/>
-      <inertia ixx="2e-5" ixy="0.0" ixz="0.0" iyy="2e-5" iyz="0.0" izz="4e-6"/>
-    </inertial>
-    <visual>
-      <origin xyz="0 0 0.0275" rpy="0 0 0"/>
-      <geometry><box size="0.012 0.010 0.055"/></geometry>
-      <material name="RG2Silver"><color rgba="0.35 0.35 0.35 1.0"/></material>
-    </visual>
-    <collision>
-      <origin xyz="0 0 0.0275" rpy="0 0 0"/>
-      <geometry><box size="0.012 0.010 0.055"/></geometry>
-    </collision>
-  </link>
-  <!-- Right finger: symmetric, moves along -Y. -->
-  <link name="rg2_rightfinger">
-    <inertial>
-      <mass value="0.040"/>
-      <origin xyz="0 0 0.0275" rpy="0 0 0"/>
-      <inertia ixx="2e-5" ixy="0.0" ixz="0.0" iyy="2e-5" iyz="0.0" izz="4e-6"/>
-    </inertial>
-    <visual>
-      <origin xyz="0 0 0.0275" rpy="0 0 0"/>
-      <geometry><box size="0.012 0.010 0.055"/></geometry>
-      <material name="RG2Silver"/>
-    </visual>
-    <collision>
-      <origin xyz="0 0 0.0275" rpy="0 0 0"/>
-      <geometry><box size="0.012 0.010 0.055"/></geometry>
-    </collision>
-  </link>
-  <!-- Pivote en Z=0.120 desde rg2_hand. Yema visual: 0.120+0.055=0.175 m desde tool0
-       (geometría visual únicamente; rg2_pinch_center semántico está en rg2_contact_tcp_xyz). -->
-  <joint name="rg2_finger_joint1" type="prismatic">
-    <parent link="rg2_hand"/>
-    <child link="rg2_leftfinger"/>
-    <origin xyz="0 0 0.120" rpy="0 0 0"/>
-    <axis xyz="0 1 0"/>
-    <limit lower="0.0" upper="0.055" effort="20" velocity="0.2"/>
-  </joint>
-  <joint name="rg2_finger_joint2" type="prismatic">
-    <parent link="rg2_hand"/>
-    <child link="rg2_rightfinger"/>
-    <origin xyz="0 0 0.120" rpy="0 0 0"/>
-    <axis xyz="0 -1 0"/>
-    <limit lower="0.0" upper="0.055" effort="20" velocity="0.2"/>
-  </joint>
-  <!-- ros2_control (gz_ros2_control) with UR5 + RG2 joints -->
-  <ros2_control name="${robot_name}" type="system">
+  <!-- ros2_control: UR5 arm joints only (no gripper). -->
+  <ros2_control name="ur5_tcp_clean" type="system">
     <hardware>
       <plugin>gz_ros2_control/GazeboSimSystem</plugin>
@@ -197,18 +124,4 @@
       <state_interface name="velocity"/>
     </joint>
-    <joint name="rg2_finger_joint1">
-      <command_interface name="position"/>
-      <state_interface name="position">
-        <param name="initial_value">0.0</param>
-      </state_interface>
-      <state_interface name="velocity"/>
-    </joint>
-    <joint name="rg2_finger_joint2">
-      <command_interface name="position"/>
-      <state_interface name="position">
-        <param name="initial_value">0.0</param>
-      </state_interface>
-      <state_interface name="velocity"/>
-    </joint>
   </ros2_control>
 </robot>

Commit message: Revert "fix(urdf): rg2_pinch_center pasa a alias explícito de rg2_tcp (B2)"
This reverts commit 26b019ec04b07df676bed54aa33bd07665962e0c.

File: agarre_ros2_ws/src/ur5_description/urdf/ur5.urdf.xacro (robot description, xacro)
@@ -80,13 +80,7 @@
     <origin xyz="${rg2_contact_tcp_xyz}" rpy="0 0 0"/>
   </joint>
-  <!-- B2 (audit 2026-05-10): rg2_pinch_center es un ALIAS explícito de rg2_tcp.
-       Históricamente eran dos frames coincidentes con mismo origin y mismo
-       parent (tool0), lo que provocaba ambigüedad semántica en el código.
-       Ahora rg2_pinch_center cuelga de rg2_tcp con transform identidad
-       (xyz=0 rpy=0), dejando inequívoco que ambos representan EL MISMO
-       punto físico (centro de cierre de la pinza RG2).
-       NO eliminamos el link/joint para preservar compatibilidad con código
-       que aún referencia rg2_pinch_center. La unificación de referencias
-       en código es deuda técnica documentada (B2 — sweep posterior). -->
+    <!-- Operational pinch-center: contact midpoint between the two RG2 fingers.
+      Keep it coincident with the semantic TCP so DIRECTO, MoveIt and attach all
+      reason about the same visible closure center. -->
   <link name="rg2_pinch_center">
     <inertial>
@@ -97,7 +91,7 @@
   </link>
   <joint name="rg2_pinch_center_joint" type="fixed">
-    <parent link="rg2_tcp"/>
+    <parent link="tool0"/>
     <child link="rg2_pinch_center"/>
-    <origin xyz="0 0 0" rpy="0 0 0"/>
+    <origin xyz="${rg2_contact_tcp_xyz}" rpy="0 0 0"/>
   </joint>
   <!-- Finger links: box 12x10x175 mm; joint origin at ±20 mm Y from rg2_base_link. -->
