Commit message: fix(tcp-geometry): unify TCP semántico rg2_pinch_center=0.0050885m en todo el stack
Corrige la geometría TCP del RG2 de forma global y elimina el valor legacy
0.175m (punta visual del dedo) que se usaba incorrectamente como offset semántico.

Cambios principales:
- urdf/ur5.urdf.xacro: rg2_contact_tcp_xyz 0.175→0.0050885; ur5_hand_joint Z/pitch
- model.sdf: anchor_joint pose 0.0050885; plugin duplicado eliminado; pitch fix
- ur5.srdf/ur5_strict.srdf: grupo end_effector declarado; pares permisivos/duplicados
  eliminados (wrist_1_link/tool0 Never, rg2_hand/wrist_2_link duplicado)
- kinematics.yaml: timeout 0.2→0.5s
- joint_limits.yaml: límites rg2 prismático [0,0.055]m
- ur5_stack.launch.py: ee_frame rg2_tcp→rg2_pinch_center (3×); tf_probe integrado
- gripper_geometry.py: guardrail Z≈0.175; patch_runtime_model_sdf usa RG2_PINCH_CENTER_FRAME
- planning_scene_sync.py: ee_frame param→rg2_pinch_center; DEFAULT_TOUCH_LINKS reordenado
- ur5_moveit_bridge.py: ee_frame param→rg2_pinch_center; ik_tip desde ee_frame
- validate_dh_vs_tf.py / find_topdown_rg2_pose.py: _PINCH_OFFSET_Z desde gripper_geometry
- inspect_rg2_visual_pose.py: constantes desde gripper_geometry
- panel_pick_demo.py / panel_pick_object.py: comentarios actualizados
- panel_runtime_pose_auditor.py / panel_settings.py: refs rg2_pinch_center
- test_gripper_geometry.py: 9 tests (guardrail + geometría canónica); 9/9 PASS
- start_panel_v2.sh: PANEL_GRIPPER_OPEN_RAD 0.5(revoluto)→0.055m(prismático)
- panel_runtime_validated.env: CLOSE_CONFIRM_TIMEOUT_SEC 120(debug)→8s(producción)

Co-Authored-By: Claude Sonnet 4.6 <noreply@anthropic.com>

File: agarre_ros2_ws/src/ur5_description/urdf/ur5.urdf.xacro (robot description, xacro)
@@ -14,7 +14,9 @@
   <xacro:property name="robot_name" value="ur5_rg2"/>
   <xacro:property name="tf_prefix_value" value=""/>
-  <!-- Offset físico real flange→yemas: 0.175 m (ur5_hand_joint Z=0.07 + finger_joint X=0.105).
-       Corregido con Opción 3 SDF fix (2026-04-24). -->
-  <xacro:property name="rg2_contact_tcp_xyz" value="0 0 0.175"/>
+  <!-- TCP semántico canónico rg2_pinch_center / rg2_tcp: 0.0050885 m desde tool0.
+       Este es el único valor válido para frames operacionales de pick, MoveIt y attach.
+       Nota: las yemas visuales de los dedos quedan a 0.120 + 0.055 = 0.175 m de tool0
+       por geometría del útil (solo relevante para visual/collision, no para TCP semántico). -->
+  <xacro:property name="rg2_contact_tcp_xyz" value="0 0 0.0050885"/>
   <xacro:property name="joint_limits_file" value="${ur_pkg_share}/config/${ur_type}/joint_limits.yaml"/>
   <xacro:property name="kinematics_file" value="${ur_pkg_share}/config/${ur_type}/default_kinematics.yaml"/>
@@ -42,21 +44,33 @@
     <origin xyz="-0.85 0 0.850" rpy="0 0 0"/>
   </xacro:ur_robot>
-  <!-- RG2 gripper (simplified kinematic stub for ros2_control) -->
-  <link name="rg2_base_link">
-    <inertial>
-      <mass value="0.5"/>
-      <origin xyz="0 0 0" rpy="0 0 0"/>
-      <inertia ixx="0.001" ixy="0.0" ixz="0.0" iyy="0.001" iyz="0.0" izz="0.001"/>
-    </inertial>
+  <!-- RG2 schematic gripper — geometry mirroring the visual_autopick_ros_ws reference.
+       rg2_hand      : gripper housing (box 60×80×120 mm), mounted at tool0.
+       rg2_leftfinger / rg2_rightfinger : thin box fingers (12×10×55 mm), prismatic ±Y.
+       Finger pivot at Z=0.120 from rg2_hand; visual tip at tool0 Z=0.175 (visual geometry only).
+       TCP semántico operacional (rg2_pinch_center) = rg2_contact_tcp_xyz = 0 0 0.0050885.
+         joint = 0.000 m → cerrada  (dedos centrados)
+         joint = 0.055 m → abierta  (cada dedo 55 mm del centro, 110 mm total) -->
+  <link name="rg2_hand">
+    <inertial>
+      <mass value="0.490"/>
+      <origin xyz="0 0 0.060" rpy="0 0 0"/>
+      <inertia ixx="0.0004" ixy="0.0" ixz="0.0" iyy="0.0004" iyz="0.0" izz="0.0003"/>
+    </inertial>
+    <visual>
+      <origin xyz="0 0 0.060" rpy="0 0 0"/>
+      <geometry><box size="0.060 0.080 0.120"/></geometry>
+      <material name="RG2Gray"><color rgba="0.18 0.18 0.18 1.0"/></material>
+    </visual>
+    <collision>
+      <origin xyz="0 0 0.060" rpy="0 0 0"/>
+      <geometry><box size="0.060 0.080 0.120"/></geometry>
+    </collision>
   </link>
   <joint name="rg2_mount_joint" type="fixed">
     <parent link="tool0"/>
-    <child link="rg2_base_link"/>
+    <child link="rg2_hand"/>
     <origin xyz="0 0 0" rpy="0 0 0"/>
   </joint>
-  <!-- Virtual TCP frame at the operational grasp center used by planning/attach.
-       The RG2 contact midpoint is slightly in front of tool0 in tool local +Z:
-       the previous -0.0877005 value landed near the finger hinges, leaving the
-       semantic TCP about 9.3 cm behind the visible pinch center. -->
+  <!-- TCP alias frame: igual que rg2_pinch_center (0 0 0.0050885 desde tool0), mantenido como alias. -->
   <link name="rg2_tcp">
     <inertial>
@@ -71,7 +85,6 @@
     <origin xyz="${rg2_contact_tcp_xyz}" rpy="0 0 0"/>
   </joint>
-    <!-- Operational pinch-center: contact midpoint between the two RG2 fingers.
-      Keep it coincident with the semantic TCP so DIRECTO, MoveIt and attach all
-      reason about the same visible closure center. -->
+  <!-- Frame operacional: 0.0050885 m desde tool0 (rg2_contact_tcp_xyz canónico).
+       TCP único usado por DIRECTO, MoveIt y el sistema attach/carry. -->
   <link name="rg2_pinch_center">
     <inertial>
@@ -86,31 +99,54 @@
     <origin xyz="${rg2_contact_tcp_xyz}" rpy="0 0 0"/>
   </joint>
-  <link name="rg2_finger_link1">
-    <inertial>
-      <mass value="0.05"/>
-      <origin xyz="0 0 0" rpy="0 0 0"/>
-      <inertia ixx="1e-4" ixy="0.0" ixz="0.0" iyy="1e-4" iyz="0.0" izz="1e-4"/>
-    </inertial>
-  </link>
-  <link name="rg2_finger_link2">
-    <inertial>
-      <mass value="0.05"/>
-      <origin xyz="0 0 0" rpy="0 0 0"/>
-      <inertia ixx="1e-4" ixy="0.0" ixz="0.0" iyy="1e-4" iyz="0.0" izz="1e-4"/>
-    </inertial>
-  </link>
+  <!-- Left finger: caja 12×10×55 mm, pivote en Z=0.120 desde rg2_hand.
+       Yema visual en Z=0.175 desde tool0 (solo geometría visual, no TCP semántico). -->
+  <link name="rg2_leftfinger">
+    <inertial>
+      <mass value="0.040"/>
+      <origin xyz="0 0 0.0275" rpy="0 0 0"/>
+      <inertia ixx="2e-5" ixy="0.0" ixz="0.0" iyy="2e-5" iyz="0.0" izz="4e-6"/>
+    </inertial>
+    <visual>
+      <origin xyz="0 0 0.0275" rpy="0 0 0"/>
+      <geometry><box size="0.012 0.010 0.055"/></geometry>
+      <material name="RG2Silver"><color rgba="0.35 0.35 0.35 1.0"/></material>
+    </visual>
+    <collision>
+      <origin xyz="0 0 0.0275" rpy="0 0 0"/>
+      <geometry><box size="0.012 0.010 0.055"/></geometry>
+    </collision>
+  </link>
+  <!-- Right finger: symmetric, moves along -Y. -->
+  <link name="rg2_rightfinger">
+    <inertial>
+      <mass value="0.040"/>
+      <origin xyz="0 0 0.0275" rpy="0 0 0"/>
+      <inertia ixx="2e-5" ixy="0.0" ixz="0.0" iyy="2e-5" iyz="0.0" izz="4e-6"/>
+    </inertial>
+    <visual>
+      <origin xyz="0 0 0.0275" rpy="0 0 0"/>
+      <geometry><box size="0.012 0.010 0.055"/></geometry>
+      <material name="RG2Silver"/>
+    </visual>
+    <collision>
+      <origin xyz="0 0 0.0275" rpy="0 0 0"/>
+      <geometry><box size="0.012 0.010 0.055"/></geometry>
+    </collision>
+  </link>
+  <!-- Pivote en Z=0.120 desde rg2_hand. Yema visual: 0.120+0.055=0.175 m desde tool0
+       (geometría visual únicamente; rg2_pinch_center semántico está en rg2_contact_tcp_xyz). -->
   <joint name="rg2_finger_joint1" type="prismatic">
-    <parent link="rg2_base_link"/>
-    <child link="rg2_finger_link1"/>
-    <origin xyz="0 0.02 0" rpy="0 0 0"/>
+    <parent link="rg2_hand"/>
+    <child link="rg2_leftfinger"/>
+    <origin xyz="0 0 0.120" rpy="0 0 0"/>
     <axis xyz="0 1 0"/>
-    <limit lower="0.0" upper="0.04" effort="20" velocity="0.2"/>
+    <limit lower="0.0" upper="0.055" effort="20" velocity="0.2"/>
   </joint>
   <joint name="rg2_finger_joint2" type="prismatic">
-    <parent link="rg2_base_link"/>
-    <child link="rg2_finger_link2"/>
-    <origin xyz="0 -0.02 0" rpy="0 0 0"/>
+    <parent link="rg2_hand"/>
+    <child link="rg2_rightfinger"/>
+    <origin xyz="0 0 0.120" rpy="0 0 0"/>
     <axis xyz="0 -1 0"/>
-    <limit lower="0.0" upper="0.04" effort="20" velocity="0.2"/>
+    <limit lower="0.0" upper="0.055" effort="20" velocity="0.2"/>
   </joint>
   <!-- ros2_control (gz_ros2_control) with UR5 + RG2 joints -->

Commit message: chore: cleanup post-defensa TFM completo (squash de 641 commits)
Squash merge de audit/fase-0-1-cleanup + 19 commits paralelos de main, tras
T35 × 5 stress live verde y borrado del path MoveIt-classic. Estado
productivo final del TFM tras aprobación.

Granularidad histórica preservada en `origin/audit/fase-0-1-cleanup` y los
6 tags publicados (ver más abajo). Squash necesario porque 2 commits viejos
de la rama main local (618564e, f93cea7) contenían .jsonl trace files
>100MB que GitHub rechaza.

=== HITOS PRINCIPALES ===

- TFM aprobado el 2026-05-08 con T35 × 3 cycles consecutivos verde live.
- Bug bloqueante BUG_CONTROLLER_FEEDBACK_HANG cerrado vía bypass
  arquitectónico (orchestrator → /pick_place → plan_to_pose_server →
  FJT directo, sin pasar por simple_controller_manager).
- Legacy `run_pick_demo` (god-closure 8.040 LOC) borrado físicamente.
- Path MoveIt-classic alternativo borrado (-17650 LOC neto):
  panel_pick_object + ur5_moveit_bridge + moveit_bridge/ mixins +
  panel_tfm_execute + direct_pick_table.
- T35 × 5 stress live verde (5/5 SUCCEEDED, media 191.2s).
- T35 × 3 post-borrado MoveIt-classic verde (3/3 SUCCEEDED, media 191.9s
  — mejor que original 214.5s).

=== REFACTOR T15 ESTRUCTURAL (2026-05-09) ===

PlanToPoseServer:
- __init__: 228 → 5 LOC con 3 helpers (_init_declare_and_read_params,
  _init_setup_tf_and_clients, _init_setup_action_server_and_bridge).
- _execute_fjt_direct: 261 → 61 LOC con 5 helpers
  (_fjt_extract_seed_positions, _fjt_compute_traj_params,
  _fjt_call_compute_ik, _fjt_build_trajectory, _fjt_send_and_wait_result).
  + Fix bug latente: seed_positions referenciado antes de definirse hacía
  que dist_to_target=0.5 SIEMPRE, forzando multi-waypoint always-on.
  Tras el fix, fases cortas usan 2-point con duration=8s — mejora -13s/cycle.
- _execute_moveit_direct: 364 → 118 LOC con 5 helpers
  (_moveit_try_fjt_bypass, _moveit_send_first_attempt,
  _moveit_post_timeout_tf_check, _moveit_retry_after_failure,
  _moveit_final_tf_recovery).

Funciones >200 LOC en plan_to_pose_server.py: 3 → 0.

=== H14 + H14b (anti-flakiness post T35×5 stress) ===

- H14 (commit e679551): fjt_direct_path_tolerance_rad=0.3rad por joint
  absorbe tracking errors transitorios sin permitir desviaciones peligrosas.
- H14b (commit c9a3aea): fjt_direct_ik_timeout_sec default 2.0→5.0s para
  tolerar latencia TRAC-IK seed-dependent post-restart.

=== FIX DUPLICATE LAUNCH ===

- start_panel_v2.sh (commit 5581967): pasar launch_plan_to_pose_server +
  launch_pick_orchestrator_lifecycle como flags. Sin esto, el panel launch
  duplicaba orchestrator + plan_to_pose_server cuando se conectaba a stack
  externo (defaults true en stack_factories.py).

=== AUDIT-V4.1 SPRINT (incorporado pre-squash) ===

19 commits separados con cleanup tier 4: env vars centralización
(panel_env, bridge_env_*), F5-iter4 mixin extraction (executor.py
1663→1491 LOC con fjt_lifecycle_mixin), schemas YAML para nodes,
mypy strict gating, etc.

=== TESTS ===

Offline: 1457 panel + 571 ur5_tools = 2028 PASSED, 0 FAILED.

Categorías: AST quality_metrics, LOC baselines, refactor T15 regresión bug
latente, FJT path tolerance, lifecycle contracts, env reads allowlist,
no_environ_drift, ui_files_loc, panel_ros_snapshot, ...

Live (sesión 10:00-11:50 UTC):
- T35 × 3 post-refactor: 206/202/196s (3/3 OK)
- T35 × 5 stress: 165.7/202.5/199.3/196.8/191.5s (5/5 OK)
- Smoke single cycle post-merge: 192.0s OK
- T35 × 3 post-borrado: 191.5/193.2/191.1s (3/3 OK)

=== TAGS PUBLICADOS EN REMOTE ===

- T35-3-cycles-verde-20260508 — criterio académico canónico (TFM aprobado)
- tfm-publicable-100-de-100-20260508 — alias publicable
- post-defensa-refactor-T15-verde-20260509 — refactor T15 verde
- tfm-t35x5-stress-verde-20260509 — T35 × 5 stress verde
- audit-pre-borrar-moveit-classic-20260509 — rollback safety pre-borrado
- tfm-cleanup-final-20260509 — cierre del cleanup
- pre-squash-main-20260509 (LOCAL) — rollback al estado merge granular

Para historial granular completo:
    git log origin/audit/fase-0-1-cleanup --oneline

Co-Authored-By: Claude Opus 4.7 (1M context) <noreply@anthropic.com>

File: agarre_ros2_ws/src/ur5_description/urdf/ur5.urdf.xacro (robot description, xacro)
@@ -14,4 +14,7 @@
   <xacro:property name="robot_name" value="ur5_rg2"/>
   <xacro:property name="tf_prefix_value" value=""/>
+  <!-- Offset físico real flange→yemas: 0.175 m (ur5_hand_joint Z=0.07 + finger_joint X=0.105).
+       Corregido con Opción 3 SDF fix (2026-04-24). -->
+  <xacro:property name="rg2_contact_tcp_xyz" value="0 0 0.175"/>
   <xacro:property name="joint_limits_file" value="${ur_pkg_share}/config/${ur_type}/joint_limits.yaml"/>
   <xacro:property name="kinematics_file" value="${ur_pkg_share}/config/${ur_type}/default_kinematics.yaml"/>
@@ -33,13 +36,26 @@
     force_abs_paths="${force_abs_paths}"
     >
-    <origin xyz="-0.85 0 0.775" rpy="0 0 0"/>
+    <!-- Keep the URDF world origin aligned with the Gazebo world include pose.
+         If these diverge, robot_state_publisher TF and the rendered Gazebo model
+         disagree in Z, which makes the panel report a different TCP height than
+         the one visible in the simulator. -->
+    <origin xyz="-0.85 0 0.850" rpy="0 0 0"/>
   </xacro:ur_robot>
-  <!-- RG2 gripper (simplified kinematic stub for ros2_control) -->
+  <!-- RG2 gripper: simplified prismatic box geometry, coherent with SDF/TF/ros2_control. -->
   <link name="rg2_base_link">
     <inertial>
-      <mass value="0.5"/>
-      <origin xyz="0 0 0" rpy="0 0 0"/>
-      <inertia ixx="0.001" ixy="0.0" ixz="0.0" iyy="0.001" iyz="0.0" izz="0.001"/>
-    </inertial>
+      <mass value="0.30"/>
+      <origin xyz="0 0 0.010" rpy="0 0 0"/>
+      <inertia ixx="0.00050" ixy="0.0" ixz="0.0" iyy="0.00040" iyz="0.0" izz="0.00060"/>
+    </inertial>
+    <visual>
+      <origin xyz="0 0 0.010" rpy="0 0 0"/>
+      <geometry><box size="0.060 0.080 0.020"/></geometry>
+      <material name="rg2_gray"><color rgba="0.4 0.4 0.4 1"/></material>
+    </visual>
+    <collision>
+      <origin xyz="0 0 0.010" rpy="0 0 0"/>
+      <geometry><box size="0.060 0.080 0.020"/></geometry>
+    </collision>
   </link>
   <joint name="rg2_mount_joint" type="fixed">
@@ -48,5 +64,8 @@
     <origin xyz="0 0 0" rpy="0 0 0"/>
   </joint>
-  <!-- Virtual TCP at the gripper fingertips (fixed offset from tool0). -->
+  <!-- Virtual TCP frame at the operational grasp center used by planning/attach.
+       The RG2 contact midpoint is slightly in front of tool0 in tool local +Z:
+       the previous -0.0877005 value landed near the finger hinges, leaving the
+       semantic TCP about 9.3 cm behind the visible pinch center. -->
   <link name="rg2_tcp">
     <inertial>
@@ -59,33 +78,68 @@
     <parent link="tool0"/>
     <child link="rg2_tcp"/>
-    <origin xyz="0 0 0.23" rpy="0 0 0"/>
-  </joint>
+    <origin xyz="${rg2_contact_tcp_xyz}" rpy="0 0 0"/>
+  </joint>
+    <!-- Operational pinch-center: contact midpoint between the two RG2 fingers.
+      Keep it coincident with the semantic TCP so DIRECTO, MoveIt and attach all
+      reason about the same visible closure center. -->
+  <link name="rg2_pinch_center">
+    <inertial>
+      <mass value="0.01"/>
+      <origin xyz="0 0 0" rpy="0 0 0"/>
+      <inertia ixx="1e-5" ixy="0.0" ixz="0.0" iyy="1e-5" iyz="0.0" izz="1e-5"/>
+    </inertial>
+  </link>
+  <joint name="rg2_pinch_center_joint" type="fixed">
+    <parent link="tool0"/>
+    <child link="rg2_pinch_center"/>
+    <origin xyz="${rg2_contact_tcp_xyz}" rpy="0 0 0"/>
+  </joint>
+  <!-- Finger links: box 12x10x175 mm; joint origin at ±20 mm Y from rg2_base_link. -->
+  <!-- Visual center at 0 0 0.0875 (half of 175 mm) in finger-link frame. -->
   <link name="rg2_finger_link1">
     <inertial>
       <mass value="0.05"/>
-      <origin xyz="0 0 0" rpy="0 0 0"/>
-      <inertia ixx="1e-4" ixy="0.0" ixz="0.0" iyy="1e-4" iyz="0.0" izz="1e-4"/>
-    </inertial>
+      <origin xyz="0 0 0.0875" rpy="0 0 0"/>
+      <inertia ixx="1.3e-4" ixy="0.0" ixz="0.0" iyy="1.3e-4" iyz="0.0" izz="1.0e-6"/>
+    </inertial>
+    <visual>
+      <origin xyz="0 0 0.0875" rpy="0 0 0"/>
+      <geometry><box size="0.012 0.010 0.175"/></geometry>
+      <material name="rg2_dark_gray"><color rgba="0.25 0.25 0.25 1"/></material>
+    </visual>
+    <collision>
+      <origin xyz="0 0 0.0875" rpy="0 0 0"/>
+      <geometry><box size="0.012 0.010 0.175"/></geometry>
+    </collision>
   </link>
   <link name="rg2_finger_link2">
     <inertial>
       <mass value="0.05"/>
-      <origin xyz="0 0 0" rpy="0 0 0"/>
-      <inertia ixx="1e-4" ixy="0.0" ixz="0.0" iyy="1e-4" iyz="0.0" izz="1e-4"/>
-    </inertial>
+      <origin xyz="0 0 0.0875" rpy="0 0 0"/>
+      <inertia ixx="1.3e-4" ixy="0.0" ixz="0.0" iyy="1.3e-4" iyz="0.0" izz="1.0e-6"/>
+    </inertial>
+    <visual>
+      <origin xyz="0 0 0.0875" rpy="0 0 0"/>
+      <geometry><box size="0.012 0.010 0.175"/></geometry>
+      <material name="rg2_dark_gray"/>
+    </visual>
+    <collision>
+      <origin xyz="0 0 0.0875" rpy="0 0 0"/>
+      <geometry><box size="0.012 0.010 0.175"/></geometry>
+    </collision>
   </link>
   <joint name="rg2_finger_joint1" type="prismatic">
     <parent link="rg2_base_link"/>
     <child link="rg2_finger_link1"/>
-    <origin xyz="0 0.02 0" rpy="0 0 0"/>
+    <origin xyz="0 0.020 0" rpy="0 0 0"/>
     <axis xyz="0 1 0"/>
-    <limit lower="0.0" upper="0.04" effort="20" velocity="0.2"/>
+    <limit lower="0.0" upper="0.0425" effort="20" velocity="0.2"/>
   </joint>
   <joint name="rg2_finger_joint2" type="prismatic">
     <parent link="rg2_base_link"/>
     <child link="rg2_finger_link2"/>
-    <origin xyz="0 -0.02 0" rpy="0 0 0"/>
+    <origin xyz="0 -0.020 0" rpy="0 0 0"/>
     <axis xyz="0 -1 0"/>
-    <limit lower="0.0" upper="0.04" effort="20" velocity="0.2"/>
+    <limit lower="0.0" upper="0.0425" effort="20" velocity="0.2"/>
   </joint>
   <!-- ros2_control (gz_ros2_control) with UR5 + RG2 joints -->
@@ -96,40 +150,56 @@
     <joint name="shoulder_pan_joint">
       <command_interface name="position"/>
-      <state_interface name="position"/>
+      <state_interface name="position">
+        <param name="initial_value">0.0</param>
+      </state_interface>
       <state_interface name="velocity"/>
     </joint>
     <joint name="shoulder_lift_joint">
       <command_interface name="position"/>
-      <state_interface name="position"/>
+      <state_interface name="position">
+        <param name="initial_value">-1.5707963267948966</param>
+      </state_interface>
       <state_interface name="velocity"/>
     </joint>
     <joint name="elbow_joint">
       <command_interface name="position"/>
-      <state_interface name="position"/>
+      <state_interface name="position">
+        <param name="initial_value">0.0</param>
+      </state_interface>
       <state_interface name="velocity"/>
     </joint>
     <joint name="wrist_1_joint">
       <command_interface name="position"/>
-      <state_interface name="position"/>
+      <state_interface name="position">
+        <param name="initial_value">-1.5707963267948966</param>
+      </state_interface>
       <state_interface name="velocity"/>
     </joint>
     <joint name="wrist_2_joint">
       <command_interface name="position"/>
-      <state_interface name="position"/>
+      <state_interface name="position">
+        <param name="initial_value">0.0</param>
+      </state_interface>
       <state_interface name="velocity"/>
     </joint>
     <joint name="wrist_3_joint">
       <command_interface name="position"/>
-      <state_interface name="position"/>
+      <state_interface name="position">
+        <param name="initial_value">0.0</param>
+      </state_interface>
       <state_interface name="velocity"/>
     </joint>
     <joint name="rg2_finger_joint1">
       <command_interface name="position"/>
-      <state_interface name="position"/>
+      <state_interface name="position">
+        <param name="initial_value">0.0</param>
+      </state_interface>
       <state_interface name="velocity"/>
     </joint>
     <joint name="rg2_finger_joint2">
       <command_interface name="position"/>
-      <state_interface name="position"/>
+      <state_interface name="position">
+        <param name="initial_value">0.0</param>
+      </state_interface>
       <state_interface name="velocity"/>
     </joint>
