Commit message: fix(urdf): rg2_pinch_center pasa a alias explícito de rg2_tcp (B2)
Cambio conservador no destructivo: rg2_pinch_center sigue existiendo
como link, pero su joint pasa a tener parent=rg2_tcp con transform
identidad (xyz=0 rpy=0) en lugar de parent=tool0 con offset 0.175.

Resuelve la ambigüedad semántica histórica donde dos frames
coincidentes pero estructuralmente independientes (mismo parent tool0,
mismo origin) confundían al código (algunos nodos usan rg2_tcp como
tip MoveIt, otros usan rg2_pinch_center como ee_frame).

Operacionalmente la TF resultante es idéntica (transform identidad),
y todo el código existente que referencia rg2_pinch_center sigue
funcionando sin cambios. La unificación de referencias en código a
rg2_tcp queda como deuda documentada (sweep posterior).

Test test_urdf_xacro_parses.py 24/24 PASS.

Bug B2 de auditoría 2026-05-10.

Co-Authored-By: Claude Opus 4.7 (1M context) <noreply@anthropic.com>

File: agarre_ros2_ws/src/ur5_description/urdf/ur5.urdf.xacro (robot description, xacro)
@@ -80,7 +80,13 @@
     <origin xyz="${rg2_contact_tcp_xyz}" rpy="0 0 0"/>
   </joint>
-    <!-- Operational pinch-center: contact midpoint between the two RG2 fingers.
-      Keep it coincident with the semantic TCP so DIRECTO, MoveIt and attach all
-      reason about the same visible closure center. -->
+  <!-- B2 (audit 2026-05-10): rg2_pinch_center es un ALIAS explícito de rg2_tcp.
+       Históricamente eran dos frames coincidentes con mismo origin y mismo
+       parent (tool0), lo que provocaba ambigüedad semántica en el código.
+       Ahora rg2_pinch_center cuelga de rg2_tcp con transform identidad
+       (xyz=0 rpy=0), dejando inequívoco que ambos representan EL MISMO
+       punto físico (centro de cierre de la pinza RG2).
+       NO eliminamos el link/joint para preservar compatibilidad con código
+       que aún referencia rg2_pinch_center. La unificación de referencias
+       en código es deuda técnica documentada (B2 — sweep posterior). -->
   <link name="rg2_pinch_center">
     <inertial>
@@ -91,7 +97,7 @@
   </link>
   <joint name="rg2_pinch_center_joint" type="fixed">
-    <parent link="tool0"/>
+    <parent link="rg2_tcp"/>
     <child link="rg2_pinch_center"/>
-    <origin xyz="${rg2_contact_tcp_xyz}" rpy="0 0 0"/>
+    <origin xyz="0 0 0" rpy="0 0 0"/>
   </joint>
   <!-- Finger links: box 12x10x175 mm; joint origin at ±20 mm Y from rg2_base_link. -->
